Commit message: Increase robot chassis length to improve stability

File: my_robot/urdf/my_robot.xacro (robot description, xacro)
@@ -8,6 +8,6 @@
     <color rgba="0.1 0.1 0.1 1"/>
   </material>
-  <material name="light_gray">
-    <color rgba="0.5 0.5 0.5 1"/>
+  <material name="white">
+    <color rgba="1 1 1 1"/>
   </material>
   <link name="robot_footprint"></link>
@@ -29,13 +29,13 @@
     </inertial>
     <collision name='chassis_collision'>
-      <origin xyz="0.05 0 0" rpy=" 0 0 0"/>
-      <geometry>
-        <box size=".25 .2 .08"/>
+      <origin xyz="0.025 0 0" rpy=" 0 0 0"/>
+      <geometry>
+        <box size=".3 .2 .08"/>
       </geometry>
     </collision>
     <visual name='chassis_visual'>
-      <origin xyz="0.05 0 0" rpy=" 0 0 0"/>
-      <geometry>
-        <box size=".25 .2 .08"/>
+      <origin xyz="0.025 0 0" rpy=" 0 0 0"/>
+      <geometry>
+        <box size=".3 .2 .08"/>
       </geometry>
       <material name="red"/>
@@ -52,8 +52,8 @@
         <box size=".1 .1 .1"/>
       </geometry>
-      <material name="light_gray"/>
+      <material name="white"/>
     </visual>
     <collision name='back_caster_collision'>
-      <origin xyz="-0.025 0 -0.05" rpy=" 0 0 0"/>
+      <origin xyz="-0.075 0 -0.05" rpy=" 0 0 0"/>
       <geometry>
         <sphere radius="0.0499"/>
@@ -61,9 +61,9 @@
     </collision>
     <visual name='back_caster_visual'>
-      <origin xyz="-0.025 0 -0.05" rpy=" 0 0 0"/>
+      <origin xyz="-0.075 0 -0.05" rpy=" 0 0 0"/>
       <geometry>
         <sphere radius="0.05"/>
       </geometry>
-      <material name="light_gray"/>
+      <material name="white"/>
     </visual>
     <collision name='front_caster_collision'>
@@ -78,5 +78,5 @@
         <sphere radius="0.05"/>
       </geometry>
-      <material name="light_gray"/>
+      <material name="white"/>
     </visual>
   </link>

Commit message: Add RGB-D camera

File: my_robot/urdf/my_robot.xacro (robot description, xacro)
@@ -176,4 +176,11 @@
     <axis xyz="0 1 0" rpy="0 0 0"/>
   </joint>
+  <joint name="camera_optical_joint" type="fixed">
+    <origin xyz="0 0 0" rpy="-1.5707 0 -1.5707"/>
+    <parent link="camera"/>
+    <child link="camera_link_optical"/>
+  </joint>
+  <link name="camera_link_optical">
+  </link>
   <link name='hokuyo'>
     <inertial>

Commit message: Implement RTAB-MAP package

File: my_robot/urdf/my_robot.xacro (robot description, xacro)
@@ -176,4 +176,6 @@
     <axis xyz="0 1 0" rpy="0 0 0"/>
   </joint>
+  <link name="camera_link_optical">
+  </link>
   <joint name="camera_optical_joint" type="fixed">
     <origin xyz="0 0 0" rpy="-1.5707 0 -1.5707"/>
@@ -181,6 +183,4 @@
     <child link="camera_link_optical"/>
   </joint>
-  <link name="camera_link_optical">
-  </link>
   <link name='hokuyo'>
     <inertial>
